Commit message: change mass value of manipulator

File: src/arm/urdf/arm.urdf (robot description, URDF)
Before this commit: robot arm, 19 links, 18 joints
Joints:
- joint l_arm_base_l_arm_link1: type fixed -> prismatic

File: src/grape_harvester/urdf/grape_harvester.urdf (robot description, URDF)
Before this commit: robot grape_harvester, 20 links, 19 joints
Links:
- removed link world
- link gripper_base: mass 0.00001 -> 0.01
- link l_arm_base: mass 0.0001 -> 0.01
- link l_arm_link_1: mass 0.00001 -> 0.01
- link l_arm_link_2: mass 0.000001 -> 0.01
- link l_arm_link_3: mass 0.000001 -> 0.01
- link l_finger_l_gripper: mass 0.00001 -> 0.01
- link r_arm_base: mass 0 -> 0.01
- link r_arm_gripper_base: mass 0.149380329868679 -> 0.01
- link r_arm_link_1: mass 0.99376961560053 -> 0.01
- link r_arm_link_2: mass 2.16979338725361 -> 0.01
- link r_arm_link_3: mass 1.51944277714983 -> 0.01
- link r_finger_l_gripper: mass 0.000001 -> 0.01
- link r_gripper_l_finger: mass 0.0155284591580667 -> 0.01
- link r_gripper_r_finger: mass 0.0162893218523249 -> 0.01
- link r_wheel_front: mass 15.911327710551 -> 15.9113277105509
Joints:
- removed joint base_joint
- joint l_arm_base_l_arm_link1: limit lower=0.3 upper=0.7 effort=300 velocity=3 -> lower=-0.2 upper=0.2 effort=300 velocity=3
- joint l_gripper_base_l_finger: origin xyz=0.15154 -0.15976 -0.083309 rpy=0 0 0.75902 -> xyz=0.151543661927759 -0.159757719126552 -0.0833093207226201 rpy=0 0 0.759018095073969
- joint l_gripper_base_r_finger: origin xyz=0.15154 -0.15976 -0.083309 rpy=0 0 0.75902 -> xyz=0.151543661927759 -0.159757719126552 -0.0833093207226201 rpy=0 0 0.759018095073969
- joint r_arm_base_r_arm_link_1: limit lower=0.3 upper=0.7 effort=300 velocity=3 -> lower=-0.2 upper=0.2 effort=300 velocity=3
