Commit message: add controller to manipulator

File: src/grape_harvester/urdf/grape_harvester.urdf (robot description, URDF)
Before this commit: robot grape_harvester, 19 links, 18 joints
Joints:
- joint l_arm_link_1_l_arm_link_2: limit lower=-3.14 upper=3.14 effort=300 velocity=3 -> lower=-2.6 upper=0.82 effort=300 velocity=3
- joint l_gripper_base_l_finger: limit lower=-0.1 upper=0.1 effort=300 velocity=3 -> lower=-0.02 upper=0 effort=300 velocity=3
- joint l_gripper_base_r_finger: limit lower=-0.1 upper=0.1 effort=300 velocity=3 -> lower=0 upper=0.02 effort=300 velocity=3
- joint r_arm_base_r_arm_link_1: origin xyz=0 0 0.455999999999899 rpy=0 0 0 -> xyz=0 0 0.593759108516829 rpy=0 0 0
- joint r_arm_link_1_r_arm_link_2: limit lower=-3.14 upper=3.14 effort=300 velocity=3 -> lower=-3.14 upper=0 effort=300 velocity=3
